File: precision clock.kicad_pcb (KiCad board)
At the start: 2 copper layers, 482.6 x 35.6 mm, 49 parts, among them J1 JACK, Q1 2N5401, Q2 2N5401, U1 MCP1700-33, X1 Crystal

Commit message: 0.56" version v1
Parts:
- removed C2: 1u, Capacitor_THT:C_Disc_D5.0mm_W2.5mm_P5.00mm
- removed C6, C7: 12p, Capacitor_THT:C_Disc_D3.0mm_W1.6mm_P2.50mm
- removed LOGO1: LOGO, precision clock:logo
- removed U1: MCP1700-33, Package_TO_SOT_THT:TO-92L_Inline_Wide
- removed X1: Crystal, Crystal:Crystal_HC18-U_Vertical
- added H1: MountingHole, MountingHole:MountingHole_3mm, F.Cu at (27.0, 127.5)
- added H2: MountingHole, MountingHole:MountingHole_3mm, F.Cu at (209.1, 127.5)
- C1: value 1u -> 100uF; footprint Capacitor_THT:C_Disc_D5.0mm_W2.5mm_P5.00mm -> Capacitor_THT:CP_Radial_D5.0mm_P2.50mm; moved to B.Cu
- C3, C4, C5: footprint Capacitor_THT:C_Disc_D3.0mm_W1.6mm_P2.50mm -> Capacitor_SMD:C_1206_3216Metric
- DCentiSec1, DCentury1, DDay1, DDecade1, DDeciSec1, DHr1, DHyphenMonth1, DHyphenYear1, DMill1, DMin1, DMonth1, DSec1, DTenDay1, DTenHr1, DTenMin1, DTenMonth1, DTenSec1, DYear1: footprint precision clock:7seg1inchCC -> precision clock:7seg0.56CC; moved to F.Cu
- DColonHM1, DColonHM2, DColonMS1, DColonMS2: footprint precision clock:LED_D3.0mm -> LED_THT:LED_D3.0mm; moved to F.Cu
- D_BST1, D_BST2, D_GMT1, D_GMT2: footprint precision clock:LED_D3.0mm -> LED_SMD:LED_1206_3216Metric; moved to F.Cu
- D_PPS1: footprint precision clock:LED_D3.0mm -> LED_SMD:LED_1206_3216Metric; moved to B.Cu
- J1, JP1, LDR1, Q1, Q2, R_Max_Bright1, R_Min_Bright1, UDateDrv1, UTimeDrv1, U_CONTROL1, U_GPS1: moved to B.Cu
- R_PPS1: footprint Resistor_THT:R_Axial_DIN0207_L6.3mm_D2.5mm_P7.62mm_Horizontal -> Resistor_SMD:R_1206_3216Metric; moved to B.Cu
- moved LDR1 482.8 mm to (22.0, 129.0), turned to 90 degrees
- moved DMill1 471.4 mm to (24.9, 127.4), turned to 0 degrees
- moved R_Min_Bright1 448.6 mm to (52.5, 130.3), turned to 90 degrees
- moved DCentury1 435.4 mm to (37.6, 127.4), turned to 0 degrees
- moved Q1 409.0 mm to (42.0, 129.5), turned to 180 degrees
- moved Q2 401.7 mm to (44.5, 129.5), turned to 0 degrees
- moved DDecade1 399.5 mm to (50.3, 127.4), turned to 0 degrees
- moved DYear1 363.7 mm to (63.0, 127.4), turned to 0 degrees
- moved R_Max_Bright1 353.9 mm to (136.5, 124.5), turned to 0 degrees
- moved DHyphenYear1 328.3 mm to (75.7, 127.4), turned to 0 degrees
- moved DTenMonth1 293.1 mm to (88.4, 127.4), turned to 0 degrees
- moved DMonth1 258.5 mm to (101.1, 127.4), turned to 0 degrees
- moved DCentiSec1 255.2 mm to (266.2, 127.4), turned to 0 degrees
- moved UDateDrv1 248.6 mm to (86.2, 130.6)
- moved DHyphenMonth1 224.5 mm to (113.8, 127.4), turned to 0 degrees
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Connections:
- C3 pad 2: /VDD_3V3 -> +5V
- DCentiSec1 pad 3: Net-(DCentiSec1-Pad3) -> unconnected-(DCentiSec1-CC-Pad3)
- DCentiSec1 pad 5: Net-(DCentiSec1-Pad5) -> unconnected-(DCentiSec1-DP-Pad5)
- DCentury1 pad 5: Net-(DCentury1-Pad5) -> unconnected-(DCentury1-DP-Pad5)
- DCentury1 pad 8: Net-(DCentury1-Pad8) -> unconnected-(DCentury1-CC-Pad8)
- DDay1 pad 5: Net-(DDay1-Pad5) -> unconnected-(DDay1-DP-Pad5)
- DDay1 pad 8: Net-(DDay1-Pad8) -> unconnected-(DDay1-CC-Pad8)
- DDecade1 pad 5: Net-(DDecade1-Pad5) -> unconnected-(DDecade1-DP-Pad5)
- DDecade1 pad 8: Net-(DDecade1-Pad8) -> unconnected-(DDecade1-CC-Pad8)
- DDeciSec1 pad 3: Net-(DDeciSec1-Pad3) -> unconnected-(DDeciSec1-CC-Pad3)
- DDeciSec1 pad 5: Net-(DDeciSec1-Pad5) -> unconnected-(DDeciSec1-DP-Pad5)
- DHr1 pad 5: Net-(DHr1-Pad5) -> unconnected-(DHr1-DP-Pad5)
- DHr1 pad 8: Net-(DHr1-Pad8) -> unconnected-(DHr1-CC-Pad8)
- DHyphenMonth1 pad 1: Net-(DHyphenMonth1-Pad1) -> unconnected-(DHyphenMonth1-E-Pad1)
- DHyphenMonth1 pad 2: Net-(DHyphenMonth1-Pad2) -> unconnected-(DHyphenMonth1-D-Pad2)
- DHyphenMonth1 pad 4: Net-(DHyphenMonth1-Pad4) -> unconnected-(DHyphenMonth1-C-Pad4)
- DHyphenMonth1 pad 5: Net-(DHyphenMonth1-Pad5) -> unconnected-(DHyphenMonth1-DP-Pad5)
- DHyphenMonth1 pad 6: Net-(DHyphenMonth1-Pad6) -> unconnected-(DHyphenMonth1-B-Pad6)
- DHyphenMonth1 pad 7: Net-(DHyphenMonth1-Pad7) -> unconnected-(DHyphenMonth1-A-Pad7)
- DHyphenMonth1 pad 8: Net-(DHyphenMonth1-Pad8) -> unconnected-(DHyphenMonth1-CC-Pad8)
- DHyphenMonth1 pad 9: Net-(DHyphenMonth1-Pad9) -> unconnected-(DHyphenMonth1-F-Pad9)
- DHyphenYear1 pad 1: Net-(DHyphenYear1-Pad1) -> unconnected-(DHyphenYear1-E-Pad1)
- DHyphenYear1 pad 2: Net-(DHyphenYear1-Pad2) -> unconnected-(DHyphenYear1-D-Pad2)
- DHyphenYear1 pad 4: Net-(DHyphenYear1-Pad4) -> unconnected-(DHyphenYear1-C-Pad4)
- DHyphenYear1 pad 5: Net-(DHyphenYear1-Pad5) -> unconnected-(DHyphenYear1-DP-Pad5)
- DHyphenYear1 pad 6: Net-(DHyphenYear1-Pad6) -> unconnected-(DHyphenYear1-B-Pad6)
- DHyphenYear1 pad 7: Net-(DHyphenYear1-Pad7) -> unconnected-(DHyphenYear1-A-Pad7)
- DHyphenYear1 pad 8: Net-(DHyphenYear1-Pad8) -> unconnected-(DHyphenYear1-CC-Pad8)
- DHyphenYear1 pad 9: Net-(DHyphenYear1-Pad9) -> unconnected-(DHyphenYear1-F-Pad9)
- DMill1 pad 5: Net-(DMill1-Pad5) -> unconnected-(DMill1-DP-Pad5)
- DMill1 pad 8: Net-(DMill1-Pad8) -> unconnected-(DMill1-CC-Pad8)
- DMin1 pad 5: Net-(DMin1-Pad5) -> unconnected-(DMin1-DP-Pad5)
- DMin1 pad 8: Net-(DMin1-Pad8) -> unconnected-(DMin1-CC-Pad8)
- DMonth1 pad 5: Net-(DMonth1-Pad5) -> unconnected-(DMonth1-DP-Pad5)
- DMonth1 pad 8: Net-(DMonth1-Pad8) -> unconnected-(DMonth1-CC-Pad8)
- DSec1 pad 8: Net-(DSec1-Pad8) -> unconnected-(DSec1-CC-Pad8)
- DTenDay1 pad 5: Net-(DTenDay1-Pad5) -> unconnected-(DTenDay1-DP-Pad5)
- DTenHr1 pad 5: Net-(DTenHr1-Pad5) -> unconnected-(DTenHr1-DP-Pad5)
- DTenHr1 pad 8: Net-(DTenHr1-Pad8) -> unconnected-(DTenHr1-CC-Pad8)
- DTenMin1 pad 5: Net-(DTenMin1-Pad5) -> unconnected-(DTenMin1-DP-Pad5)
- DTenMin1 pad 8: Net-(DTenMin1-Pad8) -> unconnected-(DTenMin1-CC-Pad8)
- DTenMonth1 pad 5: Net-(DTenMonth1-Pad5) -> unconnected-(DTenMonth1-DP-Pad5)
- DTenMonth1 pad 8: Net-(DTenMonth1-Pad8) -> unconnected-(DTenMonth1-CC-Pad8)
- DTenSec1 pad 5: Net-(DTenSec1-Pad5) -> unconnected-(DTenSec1-DP-Pad5)
- DTenSec1 pad 8: Net-(DTenSec1-Pad8) -> unconnected-(DTenSec1-CC-Pad8)
- DYear1 pad 5: Net-(DYear1-Pad5) -> unconnected-(DYear1-DP-Pad5)
- DYear1 pad 8: Net-(DYear1-Pad8) -> unconnected-(DYear1-CC-Pad8)
- R_Max_Bright1 pad 3: Net-(R_Max_Bright1-Pad3) -> unconnected-(R_Max_Bright1-Pad3)
- UDateDrv1 pad 24: Net-(UDateDrv1-Pad24) -> unconnected-(UDateDrv1-DOUT-Pad24)
- UTimeDrv1 pad 24: Net-(UTimeDrv1-Pad24) -> unconnected-(UTimeDrv1-DOUT-Pad24)
- U_CONTROL1 pad 1: Net-(U_CONTROL1-Pad1) -> unconnected-(U_CONTROL1-PA2(~{RESET}/dW/PCINT10)-Pad1)
- U_CONTROL1 pad 16: Net-(U_CONTROL1-Pad16) -> unconnected-(U_CONTROL1-(PCINT4/OC1B)PB4-Pad16)
- U_CONTROL1 pad 17: Net-(U_CONTROL1-Pad17) -> unconnected-(U_CONTROL1-(PCINT5/MOSI/DI/SDA)PB5-Pad17)
- U_CONTROL1 pad 18: Net-(U_CONTROL1-Pad18) -> unconnected-(U_CONTROL1-(PCINT6/MISO/DO)PB6-Pad18)
- U_CONTROL1 pad 19: Net-(U_CONTROL1-Pad19) -> unconnected-(U_CONTROL1-(PCINT7/USCK/SCK/SCL)PB7-Pad19)
- U_CONTROL1 pad 20: /VDD_3V3 -> +5V
- U_CONTROL1 pad 3: Net-(U_CONTROL1-Pad3) -> unconnected-(U_CONTROL1-(PCINT12/TXD)PD1-Pad3)
- U_CONTROL1 pad 4: Net-(C6-Pad2) -> unconnected-(U_CONTROL1-PA1(XTAL2/PCINT9)-Pad4)
- U_CONTROL1 pad 5: Net-(C7-Pad1) -> unconnected-(U_CONTROL1-PA0(XTAL1/CLKI/PCINT8)-Pad5)
- U_CONTROL1 pad 7: Net-(U_CONTROL1-Pad7) -> unconnected-(U_CONTROL1-(PCINT14/INT1)PD3-Pad7)
- U_CONTROL1 pad 8: Net-(U_CONTROL1-Pad8) -> unconnected-(U_CONTROL1-(PCINT15/T0)PD4-Pad8)
- U_CONTROL1 pad 9: Net-(U_CONTROL1-Pad9) -> unconnected-(U_CONTROL1-(PCINT16/OC0B/T1)PD5-Pad9)
- U_GPS1 pad 2: Net-(U_GPS1-Pad2) -> unconnected-(U_GPS1-RX-Pad2)
- U_GPS1 pad 5: /VDD_3V3 -> +5V
Routing:
- net /VDD_3V3: track 205.3 -> 0.00 mm, vias 1 -> 0
- net Net-(LDR1-Pad2): track 18.6 -> 207.7 mm, vias 0 -> 1
- net GND: track 0.00 -> 172.1 mm, vias 104 -> 10
- net Net-(D_PPS1-A): track 213.0 -> 62.8 mm, vias 0 -> 1
- net /dateA: track 258.8 -> 132.6 mm
- net /GPS_DATA: track 193.6 -> 77.5 mm
- net Net-(UDateDrv1-DIG_7): track 155.9 -> 47.5 mm, vias 0 -> 1
- net /timeD: track 255.9 -> 148.2 mm, vias 1 -> 0
- net /dateB: track 244.2 -> 138.2 mm
- net /ISET_TIME: track 297.1 -> 197.7 mm, vias 1 -> 3
- net /dateDP: track 203.4 -> 104.7 mm, vias 0 -> 2
- net /timeF: track 228.8 -> 132.8 mm
- net Net-(UDateDrv1-DIG_6): track 140.2 -> 45.0 mm, vias 1 -> 0
- net /timeC: track 260.9 -> 169.6 mm, vias 2 -> 0
- net /timeE: track 243.1 -> 153.1 mm, vias 0 -> 1
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Other:
- board size 482.6 x 35.6 mm -> 257 x 22 mm
- board text added: "0.56{dblquote} Version 2025"
- board text added: "DST"
- board text added: "Standard"
- board text removed: "(optional)"
- board text removed: "+"
- board text removed: "-"
- board text removed: "5V"
- board text removed: "GPS"
- board text removed: "Rev. 3b"
- board text removed: "Tim Jacobs and Tom Spurling, 2018"
- board text removed: "XTAL 8MHz (optional)"

Commit message: Add jumpers for permaDST and UTC
Parts:
- added JP2: Jumper_2_Open, Connector_PinHeader_2.54mm:PinHeader_1x02_P2.54mm_Vertical, B.Cu at (153.0, 136.5)
- added JP3: Jumper_2_Open, Connector_PinHeader_2.54mm:PinHeader_1x02_P2.54mm_Vertical, B.Cu at (150.5, 130.0)
- C3, C4, C5: value 100n -> 0.1uF; moved to B.Cu
- J1: value JACK -> 5V; footprint precision clock:BarrelJack_2 -> Connector_BarrelJack:BarrelJack_Horizontal
- JP1: value Jumper -> Jumper_2_Open
- moved C4 16.5 mm to (258.0, 123.0), turned to 0 degrees
- moved C3 9.71 mm to (186.5, 120.5), turned to 180 degrees
- moved J1 0.11 mm to (268.0, 124.0), turned to 90 degrees
Connections:
- U_CONTROL1 pad 4: unconnected-(U_CONTROL1-PA1(XTAL2/PCINT9)-Pad4) -> Net-(JP3-A)
- U_CONTROL1 pad 5: unconnected-(U_CONTROL1-PA0(XTAL1/CLKI/PCINT8)-Pad5) -> Net-(JP2-A)
Routing:
- net GND: track 172.1 -> 133.6 mm, vias 10 -> 24
- net Net-(JP3-A): track 0.00 -> 27.0 mm
- net Net-(JP2-A): track 0.00 -> 21.2 mm
- net +5V: track 283.5 -> 295.7 mm, vias 5 -> 7
- net /LD_TIME: track 66.2 -> 69.6 mm
- net /SPI_DATA: track 182.2 -> 179.1 mm
- net Net-(DColonMS1-K): track 66.9 -> 64.0 mm
- net /GPS_DATA: track 77.5 -> 78.7 mm
- net Net-(UTimeDrv1-DIG_6): track 70.6 -> 71.6 mm
- net Net-(D_PPS1-A): track 62.8 -> 62.3 mm
Other:
- board text added: "Brightness"
- board text added: "Enable DST"
- board text added: "Force DST"
- board text added: "GPS"
- board text added: "UTC"
- board text removed: "BRIGHTNESS"
- board text removed: "DST ENABLE"
- board text removed: "GPS FIX"
